File: PCB_Kicad/main/main.kicad_pcb (KiCad board)
At the start: 2 copper layers, 10 parts, among them U1 LT1074HV, X1 LT1006

Commit message: kicad drawings update
Parts:
- removed J_Battery1: Conn_01x02_Female, Connector_PinHeader_2.54mm:PinHeader_1x02_P2.54mm_Vertical
- removed X1: LT1006, LT1006:S8
- added C3: C_Small, Capacitor_SMD:CP_Elec_6.3x7.7, F.Cu at (191.8, 71.3)
- added C4: C_Small, Capacitor_SMD:CP_Elec_6.3x7.7, F.Cu at (182.7, 50.8)
- added C5: C_Small, Capacitor_SMD:C_1206_3216Metric, F.Cu at (163.8, 67.3)
- added C6: C_Small, Capacitor_SMD:CP_Elec_6.3x7.7, F.Cu at (148.6, 27.8)
- added D1: DIODE, Diode_SMD:D_SMC, F.Cu at (194.3, 38.1)
- added D2: DIODE, Diode_SMD:D_SMB, F.Cu at (148.5, 35.8)
- added D3: DIODE, Diode_SMD:D_SMB, F.Cu at (163.4, 52.1)
- added D_A1: D_Small, Diode_SMD:D_SMB, F.Cu at (123.2, 16.5)
- added D_A2: D_Small, Diode_SMD:D_SMB, F.Cu at (123.2, 27.8)
- added D_B1: D_Small, Diode_SMD:D_SMB, F.Cu at (130.8, 16.5)
- added D_B2: D_Small, Diode_SMD:D_SMB, F.Cu at (130.8, 27.9)
- added D_C1: D_Small, Diode_SMD:D_SMB, F.Cu at (138.4, 16.5)
- added D_C2: D_Small, Diode_SMD:D_SMB, F.Cu at (138.4, 28.2)
- added D_Ref1: D_Zener_Small, Diode_SMD:D_SOD-128, F.Cu at (184.2, 70.8)
- added D_out1: D_Schottky, Diode_SMD:D_SMB, F.Cu at (193.0, 21.3)
- added J_Bat1: Conn_01x02_Female, TerminalBlock:TerminalBlock_Altech_AK300-2_P5.00mm, F.Cu at (204.5, 21.5)
- added J_Motor1: Conn_01x03_Male, TerminalBlock:TerminalBlock_Altech_AK300-3_P5.00mm, F.Cu at (109.2, 40.6)
- added PS1: IA2412S, Converter_DCDC:Converter_DCDC_XP_POWER-IAxxxxS_THT, F.Cu at (209.6, 27.9)
- added Q1: Q_NMOS_GDS, Package_TO_SOT_THT:TO-220-3_Vertical, F.Cu at (134.6, 58.4)
- added R10: R_Small_US, Resistor_SMD:R_1206_3216Metric, F.Cu at (203.2, 57.3)
- added R11: R_Small_US, Resistor_SMD:R_1206_3216Metric, F.Cu at (207.0, 68.8)
- added R12: R_Small_US, Resistor_SMD:R_1206_3216Metric, F.Cu at (207.0, 52.1)
- added R13: R_Small_US, Resistor_SMD:R_1206_3216Metric, F.Cu at (203.2, 52.1)
- added R14: R_Small_US, Resistor_SMD:R_1206_3216Metric, F.Cu at (196.8, 50.8)
- added R15: R_Small_US, Resistor_SMD:R_1206_3216Metric, F.Cu at (189.2, 57.3)
- added R16: R_Small_US, Resistor_SMD:R_1206_3216Metric, F.Cu at (170.2, 59.7)
- added R17: R_Small_US, Resistor_SMD:R_1206_3216Metric, F.Cu at (156.2, 62.0)
- added R4: R_Small_US, Resistor_SMD:R_1206_3216Metric, F.Cu at (203.2, 62.2)
- added R5: R_Small_US, Resistor_SMD:R_1206_3216Metric, F.Cu at (191.6, 50.8)
- added R6: R_Small_US, Resistor_SMD:R_1206_3216Metric, F.Cu at (189.2, 62.2)
- added R7: R_Small_US, Resistor_SMD:R_1206_3216Metric, F.Cu at (175.3, 52.1)
- added R8: R_Small_US, Resistor_SMD:R_1206_3216Metric, F.Cu at (175.3, 57.0)
- added R9: R_Small_US, Resistor_SMD:R_1206_3216Metric, F.Cu at (175.3, 62.2)
- added REF**: Pin_D1.4mm_L8.5mm_W2.8mm_FlatFork, Connector_Pin:Pin_D1.4mm_L8.5mm_W2.8mm_FlatFork, F.Cu at (208.8, 74.2)
- added REF**: Pin_D1.4mm_L8.5mm_W2.8mm_FlatFork, Connector_Pin:Pin_D1.4mm_L8.5mm_W2.8mm_FlatFork, F.Cu at (192.5, 14.7)
- added REF**: Pin_D1.4mm_L8.5mm_W2.8mm_FlatFork, Connector_Pin:Pin_D1.4mm_L8.5mm_W2.8mm_FlatFork, F.Cu at (108.0, 17.8)
- added REF**: Pin_D1.4mm_L8.5mm_W2.8mm_FlatFork, Connector_Pin:Pin_D1.4mm_L8.5mm_W2.8mm_FlatFork, F.Cu at (108.0, 71.1)
- added REF**: Heatsink_Fischer_SK129-STS_42x25mm_2xDrill2.5mm, Heatsink:Heatsink_Fischer_SK129-STS_42x25mm_2xDrill2.5mm, F.Cu at (130.2, 55.9)
- added RV1: R_POT_TRIM_US, Potentiometer_SMD:Potentiometer_Bourns_3314G_Vertical, F.Cu at (200.7, 71.1)
- added R_Gate1: R_Small_US, Resistor_SMD:R_1206_3216Metric, F.Cu at (158.0, 39.8)
- added R_Gate2: R_Small_US, Resistor_SMD:R_1206_3216Metric, F.Cu at (154.8, 39.7)
- added U2: TL084, Package_SO:SOIC-14_3.9x8.7mm_P1.27mm, F.Cu at (182.9, 59.7)
- added U3: NA555D, Package_SO:SOIC-8_3.9x4.9mm_P1.27mm, F.Cu at (163.8, 60.3)
- added U4: FAN7371, Package_SO:SOIC-8_3.9x4.9mm_P1.27mm, F.Cu at (148.5, 41.0)
- C1: value 470uF -> 1mF; footprint Capacitor_THT:CP_Radial_D16.0mm_P7.50mm -> Capacitor_THT:CP_Radial_D8.0mm_P2.50mm
- C2: value 100nf -> 100uF; footprint Capacitor_THT:C_Rect_L7.0mm_W2.5mm_P5.00mm -> Capacitor_SMD:CP_Elec_6.3x7.7
- L1: value 100uH -> L; footprint Inductor_SMD:L_12x12mm_H8mm -> Inductor_THT:L_Radial_D29.8mm_P28.80mm_muRATA_1400series
- R1: value 10k -> R_Small_US; footprint Resistor_THT:R_Axial_DIN0207_L6.3mm_D2.5mm_P10.16mm_Horizontal -> Resistor_SMD:R_1206_3216Metric
- R2: value 100k -> R_Small_US; footprint Resistor_THT:R_Axial_DIN0207_L6.3mm_D2.5mm_P10.16mm_Horizontal -> Resistor_SMD:R_1206_3216Metric
- R3: value 2.7k -> R_Small_US; footprint Resistor_THT:R_Axial_DIN0207_L6.3mm_D2.5mm_P10.16mm_Horizontal -> Resistor_SMD:R_1206_3216Metric
- R_sense1: value 0.1R -> R_Small_US; footprint Resistor_THT:R_Axial_DIN0207_L6.3mm_D2.5mm_P10.16mm_Horizontal -> Resistor_SMD:R_1206_3216Metric
- U1: value LT1074HV -> TL084; footprint Package_TO_SOT_THT:TO-220-5_P3.4x3.7mm_StaggerOdd_Lead3.8mm_Vertical -> Package_SO:SOIC-14_3.9x8.7mm_P1.27mm
- moved R3 152.7 mm to (207.0, 62.2)
- moved U1 143.1 mm to (196.9, 59.7), turned to 180 degrees
- moved R2 136.9 mm to (207.0, 57.1)
- moved R_sense1 118.5 mm to (201.9, 30.7)
- moved R1 117.1 mm to (179.1, 71.1), turned to 90 degrees
- moved L1 100.1 mm to (173.0, 14.2), turned to 270 degrees
- moved C1 99.4 mm to (193.0, 26.7)
- moved C2 93.7 mm to (148.6, 17.6), turned to 270 degrees
Connections:
- C1 pad 2: Net-(C1-Pad2) -> GND
- C2 pad 2: 0 -> GND
- L1 pad 1: Net-(L1-Pad1) -> Net-(C1-Pad1)
- L1 pad 2: Net-(C1-Pad1) -> Net-(C6-Pad2)
- R1 pad 1: Net-(R1-Pad1) -> Net-(D_Ref1-Pad1)
- R1 pad 2: 0 -> +12V
- R2 pad 1: Net-(R1-Pad1) -> GND
- R3 pad 1: Net-(R3-Pad1) -> GND
- R3 pad 2: Net-(C2-Pad1) -> Net-(R3-Pad2)
- R_sense1 pad 1: Net-(J_Battery1-Pad2) -> V_sense
- R_sense1 pad 2: Net-(C1-Pad2) -> GND
- U1 pad 1: Net-(R2-Pad2) -> Net-(R11-Pad1)
- U1 pad 2: Net-(R3-Pad1) -> Net-(R10-Pad2)
- U1 pad 3: 0 -> V_sense
- U1 pad 4: Net-(L1-Pad1) -> +12V
- U1 pad 5: V_in -> Net-(R3-Pad2)
Routing:
- net GND: track 0.00 -> 429.3 mm
- net +12V: track 0.00 -> 160.8 mm, vias 0 -> 5
- net Net-(C6-Pad2): track 0.00 -> 106.6 mm
- net Net-(C2-Pad1): track 5.08 -> 87.8 mm, vias 0 -> 1
- net Net-(D_C1-Pad2): track 0.00 -> 59.7 mm, vias 0 -> 2
- net -12V: track 0.00 -> 54.1 mm, vias 0 -> 2
- net Net-(R11-Pad1): track 0.00 -> 53.2 mm
- net V_sense: track 0.00 -> 50.6 mm, vias 0 -> 1
- net Net-(D_B1-Pad2): track 0.00 -> 50.1 mm, vias 0 -> 2
- net PWM_Gen: track 0.00 -> 48.9 mm, vias 0 -> 2
- net PWM_REF: track 0.00 -> 43.7 mm
- net Net-(D_A1-Pad2): track 0.00 -> 41.0 mm
- net Net-(J_Battery1-Pad2): track 38.0 -> 0.00 mm
- net Net-(Q1-Pad1): track 0.00 -> 32.9 mm, vias 0 -> 1
- net Net-(R15-Pad1): track 0.00 -> 31.4 mm
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Other:
- board outline added: 111.8 x 65.4 mm
- net class Default: clearance 0.2 -> 0.25; via_drill 0.4 -> 0.45
- rule trace_clearance: 0.2 -> 0.25
