File: PCB_Kicad/main/main.sch (KiCad schematic (older format))
At the start: 10 parts, among them U1 LT1074HV, X1 LT1006

Commit message: kicad drawings update
Parts:
- removed C1: 470uF, Capacitor_THT:CP_Radial_D16.0mm_P7.50mm, symbol pspice:C
- removed C2: 100nf, Capacitor_THT:C_Rect_L7.0mm_W2.5mm_P5.00mm, symbol pspice:C
- removed J_Battery1: Conn_01x02_Female, Connector_PinHeader_2.54mm:PinHeader_1x02_P2.54mm_Vertical, symbol Connector:Conn_01x02_Female
- removed L1: 100uH, Inductor_SMD:L_12x12mm_H8mm, symbol pspice:INDUCTOR
- removed R1: 10k, Resistor_THT:R_Axial_DIN0207_L6.3mm_D2.5mm_P10.16mm_Horizontal, symbol Device:R
- removed R2: 100k, Resistor_THT:R_Axial_DIN0207_L6.3mm_D2.5mm_P10.16mm_Horizontal, symbol Device:R
- removed R3: 2.7k, Resistor_THT:R_Axial_DIN0207_L6.3mm_D2.5mm_P10.16mm_Horizontal, symbol Device:R
- removed R_sense1: 0.1R, Resistor_THT:R_Axial_DIN0207_L6.3mm_D2.5mm_P10.16mm_Horizontal, symbol Device:R
- removed U1: LT1074HV, Package_TO_SOT_THT:TO-220-5_P3.4x3.7mm_StaggerOdd_Lead3.8mm_Vertical, symbol Regulator_Switching:LT1074HV
- removed X1: LT1006, LT1006:S8, symbol LT1006:LT1006
- added C1: 1mF, Capacitor_THT:CP_Radial_D8.0mm_P2.50mm, symbol Device:C_Small
- added C2: 100uF, Capacitor_SMD:CP_Elec_6.3x7.7, symbol Device:C_Small
- added C3, C4, C6: C_Small, Capacitor_SMD:CP_Elec_6.3x7.7, symbol Device:C_Small
- added C5: C_Small, Capacitor_SMD:C_1206_3216Metric, symbol Device:C_Small
- added D1: DIODE, Diode_SMD:D_SMC, symbol Simulation_SPICE:DIODE
- added D2, D3: DIODE, Diode_SMD:D_SMB, symbol Simulation_SPICE:DIODE
- added D_A1, D_A2, D_B1, D_B2, D_C1, D_C2: D_Small, Diode_SMD:D_SMB, symbol Device:D_Small
- added D_Ref1: D_Zener_Small, Diode_SMD:D_SOD-128, symbol Device:D_Zener_Small
- added D_out1: D_Schottky, Diode_SMD:D_SMB, symbol Device:D_Schottky
- added J_Bat1: Conn_01x02_Female, TerminalBlock:TerminalBlock_Altech_AK300-2_P5.00mm, symbol Connector:Conn_01x02_Female
- added J_Motor1: Conn_01x03_Male, TerminalBlock:TerminalBlock_Altech_AK300-3_P5.00mm, symbol Connector:Conn_01x03_Male
- added L1: L, Inductor_THT:L_Radial_D29.8mm_P28.80mm_muRATA_1400series, symbol Device:L
- added PS1: IA2412S, Converter_DCDC:Converter_DCDC_XP_POWER-IAxxxxS_THT, symbol Converter_DCDC:IA2412S
- added Q1: Q_NMOS_GDS, Package_TO_SOT_THT:TO-220-3_Vertical, symbol Device:Q_NMOS_GDS
- added R1, R10, R11, R12, R13, R14, R15, R16, R17, R2, R3, R4, R5, R6, R7, R8, R9, R_Gate1, R_Gate2, R_sense1: R_Small_US, Resistor_SMD:R_1206_3216Metric, symbol Device:R_Small_US
- added RV1: R_POT_TRIM_US, Potentiometer_SMD:Potentiometer_Bourns_3314G_Vertical, symbol Device:R_POT_TRIM_US
- added U1, U2: TL084, Package_SO:SOIC-14_3.9x8.7mm_P1.27mm, symbol Amplifier_Operational:TL084
- added U3: NA555D, Package_SO:SOIC-8_3.9x4.9mm_P1.27mm, symbol Timer:NA555D
- added U4: FAN7371, Package_SO:SOIC-8_3.9x4.9mm_P1.27mm, symbol Driver_FET:FAN7371
Connections:
- net labels added: +12V, -12V, GND, PWM_Gen, PWM_REF, V_Bat, V_sense
- net labels removed: +24v, 0, V_in
- wire segments 40 -> 187

Commit message: ic tested
Parts:
- removed D1: DIODE, Diode_SMD:D_SMC, symbol Simulation_SPICE:DIODE
- removed D2, D3: DIODE, Diode_SMD:D_SMB, symbol Simulation_SPICE:DIODE
- removed D_Ref1: D_Zener_Small, Diode_SMD:D_SOD-128, symbol Device:D_Zener_Small
- removed PS1: IA2412S, Converter_DCDC:Converter_DCDC_XP_POWER-IAxxxxS_THT, symbol Converter_DCDC:IA2412S
- removed R1, R10, R11, R12, R13, R14, R15, R16, R17, R2, R3, R4, R5, R6, R7, R8, R9, R_Gate1, R_Gate2, R_sense1: R_Small_US, Resistor_SMD:R_1206_3216Metric, symbol Device:R_Small_US
- removed RV1: R_POT_TRIM_US, Potentiometer_SMD:Potentiometer_Bourns_3314G_Vertical, symbol Device:R_POT_TRIM_US
- removed U1, U2: TL084, Package_SO:SOIC-14_3.9x8.7mm_P1.27mm, symbol Amplifier_Operational:TL084
- removed U3: NA555D, Package_SO:SOIC-8_3.9x4.9mm_P1.27mm, symbol Timer:NA555D
- removed U4: FAN7371, Package_SO:SOIC-8_3.9x4.9mm_P1.27mm, symbol Driver_FET:FAN7371
- added D_Boost1: D_Small, Diode_SMD:D_SMB, symbol Device:D_Small
- added Q2: Q_NMOS_GDS, Package_TO_SOT_THT:TO-220-3_Vertical, symbol Device:Q_NMOS_GDS
- added U1: LTC3854EMSEPBF, Package_SO:MSOP-12-1EP_3x4mm_P0.65mm_EP1.65x2.85mm, symbol Regulator_Switching:LTC3854EMSEPBF
- added U2: ACS70331EESATR-005U3, Package_SO:SOIC-8-1EP_3.9x4.9mm_P1.27mm_EP2.29x3mm, symbol Sensor_Current:ACS70331EESATR-005U3
- C1: value 1mF -> 680uF; footprint Capacitor_THT:CP_Radial_D8.0mm_P2.50mm -> Capacitor_SMD:CP_Elec_6.3x7.7
- C2: value 100uF -> 68uF
- C3: value C_Small -> 2.2nF; footprint Capacitor_SMD:CP_Elec_6.3x7.7 -> Capacitor_SMD:C_1206_3216Metric
- C4: value C_Small -> 2nF; footprint Capacitor_SMD:CP_Elec_6.3x7.7 -> Capacitor_SMD:C_1206_3216Metric
- C5: value C_Small -> 1uF; footprint Capacitor_SMD:C_1206_3216Metric -> Capacitor_SMD:CP_Elec_6.3x7.7
- C6: value C_Small -> 68uF
- L1: value L -> 100uH; footprint Inductor_THT:L_Radial_D29.8mm_P28.80mm_muRATA_1400series -> Inductor_THT:L_Radial_D14.2mm_P10.00mm_Neosid_SD14
Connections:
- net GND: now also C4.2, C6.2, Q2.3 (S), U1.11 (SENSE-), U1.12 (SENSE+), U1.7 (GND), U2.3 (IP-), U2.4 (IP-), U2.5 (GND); no longer C5.1
- net V_Bat: now also D_Boost1.2 (A), U1.10 (VIN)
- net V_sense: now also U2.1 (IP+), U2.2 (IP+)
- net TG: now reaches Q1.1 (G)
- net TG: now also U1.5 (TG)
- net at C2.1, D_A1.1 (K), D_B1.1 (K)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: now also C6.1
- net SW: now reaches L1.2, Q1.3 (S)
- net SW: now also C5.1, Q2.2 (D), U1.6 (SW); no longer C6.2
- net at C3.1: now also U1.2 (ITH)
- net at C4.1: now also U1.3 (RUN/SS)
- net PWM_REF: no longer names the net of C5.2
- net PWM_REF: now also D_Boost1.1 (K), U1.4 (BOOST)
- new net +5V: U1.9 (INTVCC), U2.8 (VCC)
- new net BG: U1.8 (BG)
- new net Bg: Q2.1 (G)
- new net FeedBack: U1.1 (FB), U2.7 (VIOUT)

Commit message: kicad update
Parts:
- L1: footprint Inductor_THT:L_Radial_D14.2mm_P10.00mm_Neosid_SD14 -> Inductor_SMD:L_Wuerth_HCM-1390
Connections:
- net Bg is gone; now on an unnamed net: Q2.1 (G)
- net +5V: no longer names the net of U1.9 (INTVCC), U2.8 (VCC)
- net BG: no longer names the net of U1.8 (BG)
Changed lines of the file:
@@
 F 0 "L1" V 6519 850 50  0000 C CNN
 F 1 "100uH" V 6610 850 50  0000 C CNN
-F 2 "Inductor_THT:L_Radial_D14.2mm_P10.00mm_Neosid_SD14" H 6700 850 50  0001 C CNN
+F 2 "Inductor_SMD:L_Wuerth_HCM-1390" H 6700 850 50  0001 C CNN
 F 3 "~" H 6700 850 50  0001 C CNN
 	1    6700 850
@@
 Wire Wire Line
 	10550 2150 10450 2150
-Text GLabel 10550 1550 2    50   Input ~ 0
-+5V
-Wire Wire Line
-	10450 1550 10550 1550
-Text GLabel 6500 3400 2    50   Input ~ 0
-+5V
 $Comp
 L power:GND #PWR0102
@@
 	6450 3650 6450 3600
 Wire Wire Line
-	6200 3400 6500 3400
-Wire Wire Line
 	6200 3100 6300 3100
 Wire Wire Line
@@
 Wire Wire Line
 	6500 3300 6200 3300
-Text GLabel 6500 3500 2    50   Input ~ 0
-BG
-Wire Wire Line
-	6200 3500 6500 3500
 Text GLabel 3300 3500 0    50   Input ~ 0
 SW
@@
 Wire Wire Line
 	5750 1150 5750 1200
-Text GLabel 6400 1600 0    50   Input ~ 0
-Bg
-Wire Wire Line
-	6400 1600 6450 1600
-Wire Wire Line
-	6450 1600 6450 1550
 Text GLabel 6100 1250 3    50   Input ~ 0
 SW
@@
 Wire Wire Line
 	4200 1700 6750 1700
+Wire Wire Line
+	6200 3500 6950 3500
+Wire Wire Line
+	6950 3500 6950 1550
+Wire Wire Line
+	6950 1550 6450 1550
+Wire Wire Line
+	11000 1550 11000 3400
+Wire Wire Line
+	11000 3400 6200 3400
+Wire Wire Line
+	10450 1550 11000 1550
 $EndSCHEMATC

Commit message: model update
Parts:
- removed D_out1: D_Schottky, Diode_SMD:D_SMB, symbol Device:D_Schottky
- added C7, C8: 4.7uF, Capacitor_SMD:C_2225_5664Metric_Pad1.80x6.60mm_HandSolder, symbol Device:C_Small
Connections:
- net GND: now also C7.2, C8.2
- net V_Bat: now also C1.1, L1.1, C7.1, C8.1
Changed lines of the file:
@@
 Connection ~ 7100 850
 Wire Wire Line
-	7100 850  7550 850
+	7100 850  7500 850
 Wire Wire Line
 	7100 850  7100 1050
@@
 	9200 950  9200 850
 Wire Wire Line
-	9200 850  7850 850
-Wire Wire Line
 	9200 1050 9200 1200
 Text GLabel 9300 1200 2    50   Input ~ 0
@@
 	9200 850  9200 800
 Connection ~ 9200 850
-$Comp
-L Device:D_Schottky D_out1
-U 1 1 6006BA40
-P 7700 850
-F 0 "D_out1" H 7700 633 50  0000 C CNN
-F 1 "D_Schottky" H 7700 724 50  0000 C CNN
-F 2 "Diode_SMD:D_SMB" H 7700 850 50  0001 C CNN
-F 3 "~" H 7700 850 50  0001 C CNN
-	1    7700 850
-	-1   0    0    1
-$EndComp
 $Comp
 L power:GND #PWR0112
@@
 Wire Wire Line
 	10450 1550 11000 1550
+$Comp
+L Device:C_Small C7
+U 1 1 5FFE17AF
+P 7500 1200
+F 0 "C7" H 7592 1246 50  0000 L CNN
+F 1 "4.7uF" H 7592 1155 50  0000 L CNN
+F 2 "Capacitor_SMD:C_2225_5664Metric_Pad1.80x6.60mm_HandSolder" H 7500 1200 50  0001 C CNN
+F 3 "~" H 7500 1200 50  0001 C CNN
+	1    7500 1200
+	1    0    0    -1
+$EndComp
+Wire Wire Line
+	7500 1100 7500 850
+Connection ~ 7500 850
+Wire Wire Line
+	7500 1300 7500 1700
+Wire Wire Line
+	7500 1700 7100 1700
+Wire Wire Line
+	7500 850  7950 850
+Wire Wire Line
+	7950 1100 7950 850
+Connection ~ 7950 850
+Wire Wire Line
+	7950 1300 7950 1700
+Wire Wire Line
+	7950 1700 7500 1700
+Connection ~ 7500 1700
+$Comp
+L Device:C_Small C8
+U 1 1 5FFE1E1F
+P 7950 1200
+F 0 "C8" H 8042 1246 50  0000 L CNN
+F 1 "4.7uF" H 8042 1155 50  0000 L CNN
+F 2 "Capacitor_SMD:C_2225_5664Metric_Pad1.80x6.60mm_HandSolder" H 7950 1200 50  0001 C CNN
+F 3 "~" H 7950 1200 50  0001 C CNN
+	1    7950 1200
+	1    0    0    -1
+$EndComp
+Wire Wire Line
+	7950 850  9200 850
 $EndSCHEMATC

Commit message: kicad_updated
Parts:
- removed C6: 68uF, Capacitor_SMD:CP_Elec_6.3x7.7, symbol Device:C_Small
- C1: footprint Capacitor_SMD:CP_Elec_6.3x7.7 -> Capacitor_SMD:CP_Elec_10x7.9
- C2: footprint Capacitor_SMD:CP_Elec_6.3x7.7 -> Capacitor_THT:CP_Radial_D18.0mm_P7.50mm
- C5: footprint Capacitor_SMD:CP_Elec_6.3x7.7 -> Capacitor_SMD:CP_Elec_8x10
- C7, C8: footprint Capacitor_SMD:C_2225_5664Metric_Pad1.80x6.60mm_HandSolder -> Capacitor_SMD:C_0805_2012Metric
Changed lines of the file:
@@
 F 0 "C1" H 7192 1196 50  0000 L CNN
 F 1 "680uF" H 7192 1105 50  0000 L CNN
-F 2 "Capacitor_SMD:CP_Elec_6.3x7.7" H 7100 1150 50  0001 C CNN
+F 2 "Capacitor_SMD:CP_Elec_10x7.9" H 7100 1150 50  0001 C CNN
 F 3 "~" H 7100 1150 50  0001 C CNN
 	1    7100 1150
@@
 F 0 "C2" H 3742 1296 50  0000 L CNN
 F 1 "68uF" H 3742 1205 50  0000 L CNN
-F 2 "Capacitor_SMD:CP_Elec_6.3x7.7" H 3650 1250 50  0001 C CNN
+F 2 "Capacitor_THT:CP_Radial_D18.0mm_P7.50mm" H 3650 1250 50  0001 C CNN
 F 3 "~" H 3650 1250 50  0001 C CNN
 	1    3650 1250
@@
 	0    -1   -1   0
 $EndComp
-Wire Wire Line
-	3650 1700 4200 1700
 Wire Wire Line
 	5950 850  6100 850
@@
 F 0 "C5" H 3492 3946 50  0000 L CNN
 F 1 "1uF" H 3492 3855 50  0000 L CNN
-F 2 "Capacitor_SMD:CP_Elec_6.3x7.7" H 3400 3900 50  0001 C CNN
+F 2 "Capacitor_SMD:CP_Elec_8x10" H 3400 3900 50  0001 C CNN
 F 3 "~" H 3400 3900 50  0001 C CNN
 	1    3400 3900
@@
 Wire Wire Line
 	3400 4200 3050 4200
-$Comp
-L Device:C_Small C6
-U 1 1 5FF1C9C9
-P 4200 1250
-F 0 "C6" H 4292 1296 50  0000 L CNN
-F 1 "68uF" H 4292 1205 50  0000 L CNN
-F 2 "Capacitor_SMD:CP_Elec_6.3x7.7" H 4200 1250 50  0001 C CNN
-F 3 "~" H 4200 1250 50  0001 C CNN
-	1    4200 1250
-	1    0    0    -1
-$EndComp
-Wire Wire Line
-	4200 1150 4200 850
-Wire Wire Line
-	3650 850  4200 850
-Connection ~ 4200 850
-Wire Wire Line
-	4200 850  5550 850
-Wire Wire Line
-	4200 1350 4200 1700
-Connection ~ 4200 1700
-Wire Wire Line
-	4200 1700 6750 1700
 Wire Wire Line
 	6200 3500 6950 3500
@@
 F 0 "C7" H 7592 1246 50  0000 L CNN
 F 1 "4.7uF" H 7592 1155 50  0000 L CNN
-F 2 "Capacitor_SMD:C_2225_5664Metric_Pad1.80x6.60mm_HandSolder" H 7500 1200 50  0001 C CNN
+F 2 "Capacitor_SMD:C_0805_2012Metric" H 7500 1200 50  0001 C CNN
 F 3 "~" H 7500 1200 50  0001 C CNN
 	1    7500 1200
@@
 F 0 "C8" H 8042 1246 50  0000 L CNN
 F 1 "4.7uF" H 8042 1155 50  0000 L CNN
-F 2 "Capacitor_SMD:C_2225_5664Metric_Pad1.80x6.60mm_HandSolder" H 7950 1200 50  0001 C CNN
+F 2 "Capacitor_SMD:C_0805_2012Metric" H 7950 1200 50  0001 C CNN
 F 3 "~" H 7950 1200 50  0001 C CNN
 	1    7950 1200
@@
 Wire Wire Line
 	7950 850  9200 850
+Wire Wire Line
+	3650 850  5550 850
+Wire Wire Line
+	3650 1700 6750 1700
 $EndSCHEMATC
